Commit message: update actuator params for new motors
Co-Authored-By: Claude Opus 5.5 <noreply@anthropic.com>

File: urdf/rp1.urdf (robot description, URDF)
Before this commit: robot rp1, 29 links, 28 joints
Joints:
- joint left_ankle_pitch_joint: limit lower=-0.78 upper=0.61 effort=70.6 velocity=21.88648 -> lower=-0.78 upper=0.61 effort=64 velocity=15.70796327
- joint left_ankle_roll_joint: limit lower=-0.26 upper=0.26 effort=70.6 velocity=21.88648 -> lower=-0.26 upper=0.26 effort=64 velocity=15.70796327
- joint left_elbow_joint: limit lower=-1.6 upper=1.24 effort=35.3 velocity=21.88648 -> lower=-1.6 upper=1.24 effort=32 velocity=15.70796327
- joint left_hip_pitch_joint: limit lower=-2.86 upper=2.86 effort=141.7 velocity=14.24192 -> lower=-2.86 upper=2.86 effort=140 velocity=13.61356817
- joint left_hip_roll_joint: limit lower=-0.74 upper=2.6 effort=141.7 velocity=14.24192 -> lower=-0.74 upper=2.6 effort=140 velocity=13.61356817
- joint left_hip_yaw_joint: limit lower=-2.76 upper=2.76 effort=141.7 velocity=14.24192 -> lower=-2.76 upper=2.76 effort=55 velocity=16.23156204
- joint left_knee_joint: limit lower=-2.83 upper=0.06 effort=141.7 velocity=14.24192 -> lower=-2.83 upper=0.06 effort=140 velocity=13.61356817
- joint left_shoulder_pitch_joint: limit lower=-3.4 upper=2.35 effort=35.3 velocity=21.88648 -> lower=-3.4 upper=2.35 effort=55 velocity=16.23156204
- joint left_shoulder_roll_joint: limit lower=-0.47 upper=2.9 effort=35.3 velocity=21.88648 -> lower=-0.47 upper=2.9 effort=32 velocity=15.70796327
- joint left_shoulder_yaw_joint: limit lower=-2.87 upper=2.87 effort=35.3 velocity=21.88648 -> lower=-2.87 upper=2.87 effort=32 velocity=15.70796327
- joint left_wrist_pitch_joint: limit lower=-1.22 upper=1.22 effort=35.3 velocity=21.88648 -> lower=-1.22 upper=1.22 effort=32 velocity=15.70796327
- joint left_wrist_roll_joint: limit lower=-2.56 upper=2.56 effort=35.3 velocity=21.88648 -> lower=-2.56 upper=2.56 effort=32 velocity=15.70796327
- joint left_wrist_yaw_joint: limit lower=-1.22 upper=1.22 effort=35.3 velocity=21.88648 -> lower=-1.22 upper=1.22 effort=32 velocity=15.70796327
- joint right_ankle_pitch_joint: limit lower=-0.78 upper=0.61 effort=70.6 velocity=21.88648 -> lower=-0.78 upper=0.61 effort=64 velocity=15.70796327
- joint right_ankle_roll_joint: limit lower=-0.26 upper=0.26 effort=70.6 velocity=21.88648 -> lower=-0.26 upper=0.26 effort=64 velocity=15.70796327
- joint right_elbow_joint: limit lower=-1.24 upper=1.6 effort=35.3 velocity=21.88648 -> lower=-1.24 upper=1.6 effort=32 velocity=15.70796327
- joint right_hip_pitch_joint: limit lower=-2.86 upper=2.86 effort=141.7 velocity=14.24192 -> lower=-2.86 upper=2.86 effort=140 velocity=13.61356817
- joint right_hip_roll_joint: limit lower=-2.6 upper=0.74 effort=141.7 velocity=14.24192 -> lower=-2.6 upper=0.74 effort=140 velocity=13.61356817
- joint right_hip_yaw_joint: limit lower=-2.76 upper=2.76 effort=141.7 velocity=14.24192 -> lower=-2.76 upper=2.76 effort=55 velocity=16.23156204
- joint right_knee_joint: limit lower=-0.06 upper=2.83 effort=141.7 velocity=14.24192 -> lower=-0.06 upper=2.83 effort=140 velocity=13.61356817
- joint right_shoulder_pitch_joint: limit lower=-2.35 upper=3.4 effort=35.3 velocity=21.88648 -> lower=-2.35 upper=3.4 effort=55 velocity=16.23156204
- joint right_shoulder_roll_joint: limit lower=-2.9 upper=0.47 effort=35.3 velocity=21.88648 -> lower=-2.9 upper=0.47 effort=32 velocity=15.70796327
- joint right_shoulder_yaw_joint: limit lower=-2.87 upper=2.87 effort=35.3 velocity=21.88648 -> lower=-2.87 upper=2.87 effort=32 velocity=15.70796327
- joint right_wrist_pitch_joint: limit lower=-1.22 upper=1.22 effort=35.3 velocity=21.88648 -> lower=-1.22 upper=1.22 effort=32 velocity=15.70796327
- joint right_wrist_roll_joint: limit lower=-2.56 upper=2.56 effort=35.3 velocity=21.88648 -> lower=-2.56 upper=2.56 effort=32 velocity=15.70796327
- joint right_wrist_yaw_joint: limit lower=-1.22 upper=1.22 effort=35.3 velocity=21.88648 -> lower=-1.22 upper=1.22 effort=32 velocity=15.70796327
- joint waist_roll_joint: limit lower=-0.7 upper=0.7 effort=141.7 velocity=14.24192 -> lower=-0.7 upper=0.7 effort=140 velocity=13.61356817
- joint waist_yaw_joint: limit lower=-2.91 upper=2.91 effort=141.7 velocity=14.24192 -> lower=-2.91 upper=2.91 effort=140 velocity=13.61356817

File: urdf/rp1_24dof.urdf (robot description, URDF)
Before this commit: robot rp1, 25 links, 24 joints
Joints:
- joint left_ankle_pitch_joint: limit lower=-0.78 upper=0.61 effort=70.6 velocity=21.88648 -> lower=-0.78 upper=0.61 effort=64 velocity=15.70796327
- joint left_ankle_roll_joint: limit lower=-0.26 upper=0.26 effort=70.6 velocity=21.88648 -> lower=-0.26 upper=0.26 effort=64 velocity=15.70796327
- joint left_elbow_joint: limit lower=-1.6 upper=1.24 effort=35.3 velocity=21.88648 -> lower=-1.6 upper=1.24 effort=32 velocity=15.70796327
- joint left_hip_pitch_joint: limit lower=-2.86 upper=2.86 effort=141.7 velocity=14.24192 -> lower=-2.86 upper=2.86 effort=140 velocity=13.61356817
- joint left_hip_roll_joint: limit lower=-0.74 upper=2.6 effort=141.7 velocity=14.24192 -> lower=-0.74 upper=2.6 effort=140 velocity=13.61356817
- joint left_hip_yaw_joint: limit lower=-2.76 upper=2.76 effort=141.7 velocity=14.24192 -> lower=-2.76 upper=2.76 effort=55 velocity=16.23156204
- joint left_knee_joint: limit lower=-2.83 upper=0.06 effort=141.7 velocity=14.24192 -> lower=-2.83 upper=0.06 effort=140 velocity=13.61356817
- joint left_shoulder_pitch_joint: limit lower=-3.4 upper=2.35 effort=35.3 velocity=21.88648 -> lower=-3.4 upper=2.35 effort=55 velocity=16.23156204
- joint left_shoulder_roll_joint: limit lower=-0.47 upper=2.9 effort=35.3 velocity=21.88648 -> lower=-0.47 upper=2.9 effort=32 velocity=15.70796327
- joint left_shoulder_yaw_joint: limit lower=-2.87 upper=2.87 effort=35.3 velocity=21.88648 -> lower=-2.87 upper=2.87 effort=32 velocity=15.70796327
- joint left_wrist_joint: limit lower=-2.56 upper=2.56 effort=35.3 velocity=21.88648 -> lower=-2.56 upper=2.56 effort=32 velocity=15.70796327
- joint right_ankle_pitch_joint: limit lower=-0.78 upper=0.61 effort=70.6 velocity=21.88648 -> lower=-0.78 upper=0.61 effort=64 velocity=15.70796327
- joint right_ankle_roll_joint: limit lower=-0.26 upper=0.26 effort=70.6 velocity=21.88648 -> lower=-0.26 upper=0.26 effort=64 velocity=15.70796327
- joint right_elbow_joint: limit lower=-1.24 upper=1.6 effort=35.3 velocity=21.88648 -> lower=-1.24 upper=1.6 effort=32 velocity=15.70796327
- joint right_hip_pitch_joint: limit lower=-2.86 upper=2.86 effort=141.7 velocity=14.24192 -> lower=-2.86 upper=2.86 effort=140 velocity=13.61356817
- joint right_hip_roll_joint: limit lower=-2.6 upper=0.74 effort=141.7 velocity=14.24192 -> lower=-2.6 upper=0.74 effort=140 velocity=13.61356817
- joint right_hip_yaw_joint: limit lower=-2.76 upper=2.76 effort=141.7 velocity=14.24192 -> lower=-2.76 upper=2.76 effort=55 velocity=16.23156204
- joint right_knee_joint: limit lower=-0.06 upper=2.83 effort=141.7 velocity=14.24192 -> lower=-0.06 upper=2.83 effort=140 velocity=13.61356817
- joint right_shoulder_pitch_joint: limit lower=-2.35 upper=3.4 effort=35.3 velocity=21.88648 -> lower=-2.35 upper=3.4 effort=55 velocity=16.23156204
- joint right_shoulder_roll_joint: limit lower=-2.9 upper=0.47 effort=35.3 velocity=21.88648 -> lower=-2.9 upper=0.47 effort=32 velocity=15.70796327
- joint right_shoulder_yaw_joint: limit lower=-2.87 upper=2.87 effort=35.3 velocity=21.88648 -> lower=-2.87 upper=2.87 effort=32 velocity=15.70796327
- joint right_wrist_joint: limit lower=-2.56 upper=2.56 effort=35.3 velocity=21.88648 -> lower=-2.56 upper=2.56 effort=32 velocity=15.70796327
- joint waist_roll_joint: limit lower=-0.7 upper=0.7 effort=141.7 velocity=14.24192 -> lower=-0.7 upper=0.7 effort=140 velocity=13.61356817
- joint waist_yaw_joint: limit lower=-2.91 upper=2.91 effort=141.7 velocity=14.24192 -> lower=-2.91 upper=2.91 effort=140 velocity=13.61356817

File: urdf/rp1_hand.urdf (robot description, URDF)
Before this commit: robot rp1, 63 links, 62 joints
Joints:
- joint left_ankle_pitch_joint: limit lower=-0.78 upper=0.61 effort=70.6 velocity=21.88648 -> lower=-0.78 upper=0.61 effort=64 velocity=15.70796327
- joint left_ankle_roll_joint: limit lower=-0.26 upper=0.26 effort=70.6 velocity=21.88648 -> lower=-0.26 upper=0.26 effort=64 velocity=15.70796327
- joint left_elbow_joint: limit lower=-1.6 upper=1.24 effort=35.3 velocity=21.88648 -> lower=-1.6 upper=1.24 effort=32 velocity=15.70796327
- joint left_hip_pitch_joint: limit lower=-2.86 upper=2.86 effort=141.7 velocity=14.24192 -> lower=-2.86 upper=2.86 effort=140 velocity=13.61356817
- joint left_hip_roll_joint: limit lower=-0.74 upper=2.6 effort=141.7 velocity=14.24192 -> lower=-0.74 upper=2.6 effort=140 velocity=13.61356817
- joint left_hip_yaw_joint: limit lower=-2.76 upper=2.76 effort=141.7 velocity=14.24192 -> lower=-2.76 upper=2.76 effort=55 velocity=16.23156204
- joint left_knee_joint: limit lower=-2.83 upper=0.06 effort=141.7 velocity=14.24192 -> lower=-2.83 upper=0.06 effort=140 velocity=13.61356817
- joint left_shoulder_pitch_joint: limit lower=-3.4 upper=2.35 effort=35.3 velocity=21.88648 -> lower=-3.4 upper=2.35 effort=55 velocity=16.23156204
- joint left_shoulder_roll_joint: limit lower=-0.47 upper=2.9 effort=35.3 velocity=21.88648 -> lower=-0.47 upper=2.9 effort=32 velocity=15.70796327
- joint left_shoulder_yaw_joint: limit lower=-2.87 upper=2.87 effort=35.3 velocity=21.88648 -> lower=-2.87 upper=2.87 effort=32 velocity=15.70796327
- joint left_wrist_pitch_joint: limit lower=-1.22 upper=1.22 effort=35.3 velocity=21.88648 -> lower=-1.22 upper=1.22 effort=32 velocity=15.70796327
- joint left_wrist_roll_joint: limit lower=-2.56 upper=2.56 effort=35.3 velocity=21.88648 -> lower=-2.56 upper=2.56 effort=32 velocity=15.70796327
- joint left_wrist_yaw_joint: limit lower=-1.22 upper=1.22 effort=35.3 velocity=21.88648 -> lower=-1.22 upper=1.22 effort=32 velocity=15.70796327
- joint right_ankle_pitch_joint: limit lower=-0.78 upper=0.61 effort=70.6 velocity=21.88648 -> lower=-0.78 upper=0.61 effort=64 velocity=15.70796327
- joint right_ankle_roll_joint: limit lower=-0.26 upper=0.26 effort=70.6 velocity=21.88648 -> lower=-0.26 upper=0.26 effort=64 velocity=15.70796327
- joint right_elbow_joint: limit lower=-1.24 upper=1.6 effort=35.3 velocity=21.88648 -> lower=-1.24 upper=1.6 effort=32 velocity=15.70796327
- joint right_hip_pitch_joint: limit lower=-2.86 upper=2.86 effort=141.7 velocity=14.24192 -> lower=-2.86 upper=2.86 effort=140 velocity=13.61356817
- joint right_hip_roll_joint: limit lower=-2.6 upper=0.74 effort=141.7 velocity=14.24192 -> lower=-2.6 upper=0.74 effort=140 velocity=13.61356817
- joint right_hip_yaw_joint: limit lower=-2.76 upper=2.76 effort=141.7 velocity=14.24192 -> lower=-2.76 upper=2.76 effort=55 velocity=16.23156204
- joint right_knee_joint: limit lower=-0.06 upper=2.83 effort=141.7 velocity=14.24192 -> lower=-0.06 upper=2.83 effort=140 velocity=13.61356817
- joint right_shoulder_pitch_joint: limit lower=-2.35 upper=3.4 effort=35.3 velocity=21.88648 -> lower=-2.35 upper=3.4 effort=55 velocity=16.23156204
- joint right_shoulder_roll_joint: limit lower=-2.9 upper=0.47 effort=35.3 velocity=21.88648 -> lower=-2.9 upper=0.47 effort=32 velocity=15.70796327
- joint right_shoulder_yaw_joint: limit lower=-2.87 upper=2.87 effort=35.3 velocity=21.88648 -> lower=-2.87 upper=2.87 effort=32 velocity=15.70796327
- joint right_wrist_pitch_joint: limit lower=-1.22 upper=1.22 effort=35.3 velocity=21.88648 -> lower=-1.22 upper=1.22 effort=32 velocity=15.70796327
- joint right_wrist_roll_joint: limit lower=-2.56 upper=2.56 effort=35.3 velocity=21.88648 -> lower=-2.56 upper=2.56 effort=32 velocity=15.70796327
- joint right_wrist_yaw_joint: limit lower=-1.22 upper=1.22 effort=35.3 velocity=21.88648 -> lower=-1.22 upper=1.22 effort=32 velocity=15.70796327
- joint waist_roll_joint: limit lower=-0.7 upper=0.7 effort=141.7 velocity=14.24192 -> lower=-0.7 upper=0.7 effort=140 velocity=13.61356817
- joint waist_yaw_joint: limit lower=-2.91 upper=2.91 effort=141.7 velocity=14.24192 -> lower=-2.91 upper=2.91 effort=140 velocity=13.61356817

File: urdf/rp1_hand_fixed.urdf (robot description, URDF)
Before this commit: robot rp1_hand_fixed, 63 links, 62 joints
Joints:
- joint left_ankle_pitch_joint: limit lower=-0.78 upper=0.61 effort=70.6 velocity=21.88648 -> lower=-0.78 upper=0.61 effort=64 velocity=15.70796327
- joint left_ankle_roll_joint: limit lower=-0.26 upper=0.26 effort=70.6 velocity=21.88648 -> lower=-0.26 upper=0.26 effort=64 velocity=15.70796327
- joint left_elbow_joint: limit lower=-1.6 upper=1.24 effort=35.3 velocity=21.88648 -> lower=-1.6 upper=1.24 effort=32 velocity=15.70796327
- joint left_hip_pitch_joint: limit lower=-2.86 upper=2.86 effort=141.7 velocity=14.24192 -> lower=-2.86 upper=2.86 effort=140 velocity=13.61356817
- joint left_hip_roll_joint: limit lower=-0.74 upper=2.6 effort=141.7 velocity=14.24192 -> lower=-0.74 upper=2.6 effort=140 velocity=13.61356817
- joint left_hip_yaw_joint: limit lower=-2.76 upper=2.76 effort=141.7 velocity=14.24192 -> lower=-2.76 upper=2.76 effort=55 velocity=16.23156204
- joint left_knee_joint: limit lower=-2.83 upper=0.06 effort=141.7 velocity=14.24192 -> lower=-2.83 upper=0.06 effort=140 velocity=13.61356817
- joint left_shoulder_pitch_joint: limit lower=-3.4 upper=2.35 effort=35.3 velocity=21.88648 -> lower=-3.4 upper=2.35 effort=55 velocity=16.23156204
- joint left_shoulder_roll_joint: limit lower=-0.47 upper=2.9 effort=35.3 velocity=21.88648 -> lower=-0.47 upper=2.9 effort=32 velocity=15.70796327
- joint left_shoulder_yaw_joint: limit lower=-2.87 upper=2.87 effort=35.3 velocity=21.88648 -> lower=-2.87 upper=2.87 effort=32 velocity=15.70796327
- joint left_wrist_pitch_joint: limit lower=-1.22 upper=1.22 effort=35.3 velocity=21.88648 -> lower=-1.22 upper=1.22 effort=32 velocity=15.70796327
- joint left_wrist_roll_joint: limit lower=-2.56 upper=2.56 effort=35.3 velocity=21.88648 -> lower=-2.56 upper=2.56 effort=32 velocity=15.70796327
- joint left_wrist_yaw_joint: limit lower=-1.22 upper=1.22 effort=35.3 velocity=21.88648 -> lower=-1.22 upper=1.22 effort=32 velocity=15.70796327
- joint right_ankle_pitch_joint: limit lower=-0.78 upper=0.61 effort=70.6 velocity=21.88648 -> lower=-0.78 upper=0.61 effort=64 velocity=15.70796327
- joint right_ankle_roll_joint: limit lower=-0.26 upper=0.26 effort=70.6 velocity=21.88648 -> lower=-0.26 upper=0.26 effort=64 velocity=15.70796327
- joint right_elbow_joint: limit lower=-1.24 upper=1.6 effort=35.3 velocity=21.88648 -> lower=-1.24 upper=1.6 effort=32 velocity=15.70796327
- joint right_hip_pitch_joint: limit lower=-2.86 upper=2.86 effort=141.7 velocity=14.24192 -> lower=-2.86 upper=2.86 effort=140 velocity=13.61356817
- joint right_hip_roll_joint: limit lower=-2.6 upper=0.74 effort=141.7 velocity=14.24192 -> lower=-2.6 upper=0.74 effort=140 velocity=13.61356817
- joint right_hip_yaw_joint: limit lower=-2.76 upper=2.76 effort=141.7 velocity=14.24192 -> lower=-2.76 upper=2.76 effort=55 velocity=16.23156204
- joint right_knee_joint: limit lower=-0.06 upper=2.83 effort=141.7 velocity=14.24192 -> lower=-0.06 upper=2.83 effort=140 velocity=13.61356817
- joint right_shoulder_pitch_joint: limit lower=-2.35 upper=3.4 effort=35.3 velocity=21.88648 -> lower=-2.35 upper=3.4 effort=55 velocity=16.23156204
- joint right_shoulder_roll_joint: limit lower=-2.9 upper=0.47 effort=35.3 velocity=21.88648 -> lower=-2.9 upper=0.47 effort=32 velocity=15.70796327
- joint right_shoulder_yaw_joint: limit lower=-2.87 upper=2.87 effort=35.3 velocity=21.88648 -> lower=-2.87 upper=2.87 effort=32 velocity=15.70796327
- joint right_wrist_pitch_joint: limit lower=-1.22 upper=1.22 effort=35.3 velocity=21.88648 -> lower=-1.22 upper=1.22 effort=32 velocity=15.70796327
- joint right_wrist_roll_joint: limit lower=-2.56 upper=2.56 effort=35.3 velocity=21.88648 -> lower=-2.56 upper=2.56 effort=32 velocity=15.70796327
- joint right_wrist_yaw_joint: limit lower=-1.22 upper=1.22 effort=35.3 velocity=21.88648 -> lower=-1.22 upper=1.22 effort=32 velocity=15.70796327
- joint waist_roll_joint: limit lower=-0.7 upper=0.7 effort=141.7 velocity=14.24192 -> lower=-0.7 upper=0.7 effort=140 velocity=13.61356817
- joint waist_yaw_joint: limit lower=-2.91 upper=2.91 effort=141.7 velocity=14.24192 -> lower=-2.91 upper=2.91 effort=140 velocity=13.61356817
