Commit message: Add RP1 white and blue visuals with shared STL assets

File: urdf/rp1.urdf (robot description, URDF)
Before this commit: robot rp1, 29 links, 28 joints
Links:
- link base_link: geometry visual mesh filename=../meshes/base_link.STL; visual mesh filename=../meshes/base_link_hip_flange_blue.STL
- link left_ankle_roll_link: geometry collision cylinder length=0.06 radius=0.01; collision cylinder length=0.06 radius=0.01
- link right_ankle_roll_link: geometry collision cylinder length=0.06 radius=0.01; collision cylinder length=0.06 radius=0.01
- link waist_yaw_link: geometry collision mesh filename=../meshes/waist_yaw_link.STL; visual mesh filename=../meshes/waist_yaw_link_visual_white.STL

File: urdf/rp1_24dof.urdf (robot description, URDF)
Before this commit: robot rp1, 25 links, 24 joints
Links:
- link base_link: geometry visual mesh filename=../meshes/base_link.STL; visual mesh filename=../meshes/base_link_hip_flange_blue.STL
- link left_ankle_roll_link: geometry collision cylinder length=0.06 radius=0.01; collision cylinder length=0.06 radius=0.01
- link right_ankle_roll_link: geometry collision cylinder length=0.06 radius=0.01; collision cylinder length=0.06 radius=0.01
- link waist_yaw_link: geometry collision mesh filename=../meshes/waist_yaw_link.STL; visual mesh filename=../meshes/waist_yaw_link_visual_white.STL

File: urdf/rp1_hand.urdf (robot description, URDF)
Before this commit: robot rp1, 63 links, 62 joints
Links:
- link base_link: geometry visual mesh filename=../meshes/base_link.STL; visual mesh filename=../meshes/base_link_hip_flange_blue.STL
- link left_ankle_roll_link: geometry collision cylinder length=0.06 radius=0.01; collision cylinder length=0.06 radius=0.01
- link right_ankle_roll_link: geometry collision cylinder length=0.06 radius=0.01; collision cylinder length=0.06 radius=0.01
- link waist_yaw_link: geometry collision mesh filename=../meshes/waist_yaw_link.STL; visual mesh filename=../meshes/waist_yaw_link_visual_white.STL

File: urdf/rp1_hand_fixed.urdf (robot description, URDF)
Before this commit: robot rp1_hand_fixed, 63 links, 62 joints
Links:
- link base_link: geometry visual mesh filename=../meshes/base_link.STL; visual mesh filename=../meshes/base_link_hip_flange_blue.STL
- link left_ankle_roll_link: geometry collision cylinder length=0.06 radius=0.01; collision cylinder length=0.06 radius=0.01
- link right_ankle_roll_link: geometry collision cylinder length=0.06 radius=0.01; collision cylinder length=0.06 radius=0.01
- link waist_yaw_link: geometry collision mesh filename=../meshes/waist_yaw_link.STL; visual mesh filename=../meshes/waist_yaw_link_visual_white.STL
